File: MRCS-ATSN.brd (EAGLE design)
At the start: 159.8 x 68.8 mm, 66 parts, among them CON1 Audio, CON2 Break-In, IC1 LM324N, IC2 LM324N, J1 RJ14, J2 RJ14, Q1 2N4401, Q2 2N4403, T1 TY-145P

Commit message: added missing values
Parts:
- CON1: value Audio -> 0.100
- CON2: value Break-In -> 0.100
- JP1, JP4, JP8, SL1, SL2, SL3: value (none) -> 0.100
- JP5: value Phase -> 0.100
Changed lines of the file:
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@@
 <attribute name="VALUE" x="99.187" y="27.94" size="1.4224" layer="27" font="vector"/>
 </element>
-<element name="JP4" library="SPCoast" package="1X02_LOCK" value="" x="57.15" y="25.4" smashed="yes" rot="R270">
+<element name="JP4" library="SPCoast" package="1X02_LOCK" value="0.100" x="57.15" y="25.4" smashed="yes" rot="R270">
 <attribute name="NAME" x="64.6938" y="26.3652" size="1.4224" layer="25" font="vector" ratio="10" rot="R270"/>
 <attribute name="VALUE" x="53.975" y="26.67" size="1.27" layer="27" rot="R270"/>
@@
 <attribute name="VALUE" x="66.5" y="14.32" size="1.4224" layer="27" font="vector" rot="R90"/>
 </element>
-<element name="JP5" library="SPCoast" package="1X03" value="Phase" x="74.93" y="31.115" smashed="yes">
+<element name="JP5" library="SPCoast" package="1X03" value="0.100" x="74.93" y="31.115" smashed="yes">
 <attribute name="NAME" x="69.6468" y="30.5308" size="1.4224" layer="25" font="vector" ratio="10"/>
 <attribute name="VALUE" x="80.645" y="34.925" size="1.4224" layer="27" font="vector" rot="R180"/>
@@
 <attribute name="VALUE" x="80.47" y="14.32" size="1.4224" layer="27" font="vector" rot="R90"/>
 </element>
-<element name="JP8" library="SPCoast" package="1X02_LOCK" value="" x="71.12" y="25.4" smashed="yes" rot="R270">
+<element name="JP8" library="SPCoast" package="1X02_LOCK" value="0.100" x="71.12" y="25.4" smashed="yes" rot="R270">
 <attribute name="NAME" x="78.6638" y="26.1112" size="1.4224" layer="25" font="vector" ratio="10" rot="R270"/>
 <attribute name="VALUE" x="67.945" y="26.67" size="1.27" layer="27" rot="R270"/>
@@
 <attribute name="VALUE" x="37.846" y="48.641" size="0.8128" layer="27" font="vector" ratio="15" rot="R180"/>
 </element>
-<element name="SL2" library="SPCoast" package="MOLEX-1X4_LOCK" value="" x="111.76" y="35.56" smashed="yes"/>
+<element name="SL2" library="SPCoast" package="MOLEX-1X4_LOCK" value="0.100" x="111.76" y="35.56" smashed="yes"/>
 <element name="JP9" library="SPCoast" package="MSTB2" value="" x="133.35" y="19.05" smashed="yes">
 <attribute name="NAME" x="132.207" y="16.637" size="1.4224" layer="25" font="vector" ratio="10"/>
 <attribute name="VALUE" x="130.4501" y="22.8501" size="0.02" layer="27"/>
 </element>
-<element name="SL1" library="SPCoast" package="MOLEX-1X4_LOCK" value="" x="92.71" y="35.56" smashed="yes"/>
+<element name="SL1" library="SPCoast" package="MOLEX-1X4_LOCK" value="0.100" x="92.71" y="35.56" smashed="yes"/>
 <element name="R1" library="bourns_test" package="3386K" value="10K" x="11.43" y="15.24" smashed="yes">
 <attribute name="NAME" x="9.2075" y="11.7475" size="1.4224" layer="25" font="vector" ratio="12"/>
@@
 </element>
 <element name="U$1" library="SPCoast" package="MRCS-LOGO" value="MRCS-LOGOBOT-LARGE" x="88.9" y="33.655" smashed="yes"/>
-<element name="SL3" library="SPCoast" package="MOLEX-1X4_LOCK" value="" x="31.75" y="24.13" smashed="yes"/>
-<element name="CON1" library="SPCoast 2017_04" package="1X04_LOCK" value="Audio" x="20.32" y="24.13" smashed="yes">
+<element name="SL3" library="SPCoast" package="MOLEX-1X4_LOCK" value="0.100" x="31.75" y="24.13" smashed="yes"/>
+<element name="CON1" library="SPCoast 2017_04" package="1X04_LOCK" value="0.100" x="20.32" y="24.13" smashed="yes">
 <attribute name="NAME" x="18.9738" y="25.9588" size="1.27" layer="25" font="vector" ratio="10"/>
 <attribute name="VALUE" x="19.05" y="20.955" size="1.27" layer="27" font="vector"/>
 </element>
-<element name="CON2" library="SPCoast 2017_04" package="1X04_LOCK" value="Break-In" x="7.62" y="24.13" smashed="yes">
+<element name="CON2" library="SPCoast 2017_04" package="1X04_LOCK" value="0.100" x="7.62" y="24.13" smashed="yes">
 <attribute name="NAME" x="6.2738" y="25.9588" size="1.27" layer="25" font="vector" ratio="10"/>
 <attribute name="VALUE" x="6.35" y="20.955" size="1.27" layer="27" font="vector"/>
@@
 <attribute name="VALUE" x="9.144" y="59.309" size="0.8128" layer="21" font="vector" ratio="15"/>
 </element>
-<element name="JP1" library="SPCoast" package="1X02_LOCK" value="" x="3.81" y="53.34" smashed="yes" rot="R90">
+<element name="JP1" library="SPCoast" package="1X02_LOCK" value="0.100" x="3.81" y="53.34" smashed="yes" rot="R90">
 <attribute name="NAME" x="1.9812" y="51.9938" size="1.27" layer="25" font="vector" ratio="10" rot="R90"/>
 <attribute name="VALUE" x="6.985" y="52.07" size="1.27" layer="27" rot="R90"/>

Commit message: added missing values
Parts:
- JP9: value (none) -> 0.200
Changed lines of the file:
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@@
 </element>
 <element name="SL2" library="SPCoast" package="MOLEX-1X4_LOCK" value="0.100" x="111.76" y="35.56" smashed="yes"/>
-<element name="JP9" library="SPCoast" package="MSTB2" value="" x="133.35" y="19.05" smashed="yes">
+<element name="JP9" library="SPCoast" package="MSTB2" value="0.200" x="133.35" y="19.05" smashed="yes">
 <attribute name="NAME" x="132.207" y="16.637" size="1.4224" layer="25" font="vector" ratio="10"/>
 <attribute name="VALUE" x="130.4501" y="22.8501" size="0.02" layer="27"/>
